File: preliminary_board/ece_411_team9_bird_feeder.brd (EAGLE design)
At the start: 160 x 100 mm, 11 parts, among them IC1 TINY13V-10PU, IC2 LM741P, IC3 LM741P, M1 ELECTRET_MICROPHON-WM.64PN, M2 SERVO

Commit message: Add files via upload
Parts:
- removed SENSOR: (no value), pinhead:1X02/90
- added C1: 0.33uF, eagle-ltspice:C0805
- added C2, C3, C4, C5: 0.1uF, eagle-ltspice:C0805
- added CN1: V_battery, adafruit:JST-PH-2-SMT
- added FORC_SENS: (no value), pinhead:1X02/90
- added IC4: 7805TV, linear:TO220V
- added R6: 100K, eagle-ltspice:R0805
- R1, R2, R3, R4: value (none) -> 10K; device eagle-ltspice:0207/10 -> eagle-ltspice:R0805
- R5: value (none) -> 1K; device eagle-ltspice:0207/10 -> eagle-ltspice:R0805
- moved R2 29.0 mm to (22.9, 14.0)
- moved R4 24.2 mm to (19.1, 19.1), turned to 0 degrees
- moved R3 18.8 mm to (16.5, 21.6)
- moved R1 4.58 mm to (11.4, 21.6)
- moved R5 2.84 mm to (45.7, 16.5)
Connections:
- net N$5 renamed MIC_INT
- removed net N$1: IC1.8, IC2.2, R1.1, R2.1, SENSOR.1
- removed net N$12: IC1.1, IC3.6, R5.1
- removed net N$2: IC2.1, IC2.5
- removed net N$3: IC3.1, IC3.5
- removed net V_BATT: IC2.7, IC3.7, R1.2
- new net 7.4V: C1.1, CN1.1, IC4.1
- new net MIC_OUT: IC1.1, IC3.6, R6.2
- new net N$8: IC2.2, R1.1, R3.2
- net +5V: now also C2.1, C3.1, C4.2, C5.1, FORC_SENS.1, IC1.8, IC2.7, IC3.7, IC4.3, R1.2, R2.2
- net GND: now also C1.2, C2.2, C3.2, C4.1, C5.2, CN1.2, IC4.2, R4.1, R5.1; no longer R2.2, R4.2
- net N$13: now also R6.1; no longer R4.1
- net N$4: now also FORC_SENS.2, R2.1, R4.2; no longer R3.2, SENSOR.2
Routing:
- net +5V: track 48.3 -> 136.5 mm, vias 3 -> 8
- net GND: track 74.9 -> 158.5 mm, vias 5 -> 12
- net N$1: track 82.6 -> 0.00 mm, vias 6 -> 0
- net 7.4V: track 0.00 -> 66.2 mm, vias 0 -> 2
- net V_BATT: track 53.9 -> 0.00 mm, vias 6 -> 0
- net N$12: track 32.4 -> 0.00 mm, vias 1 -> 0
- net MIC_OUT: track 0.00 -> 27.1 mm, vias 0 -> 1
- net N$2: track 15.2 -> 0.00 mm, vias 2 -> 0
- net N$8: track 0.00 -> 11.8 mm
- net N$3: track 10.8 -> 0.00 mm
- net N$13: track 25.1 -> 18.4 mm, vias 1 -> 3
- net N$9: track 14.7 -> 12.5 mm
- net N$4: track 31.8 -> 29.6 mm, vias 1 -> 2
- net MIC_INT: track 30.9 -> 30.3 mm
- added copper zone on layer 1, net GND
Other:
- board text added: "Bird Feeder Board Rev 1.0"
- board text removed: "FA20 ECE 411 - Team 9: Preliminary Board"

Commit message: Add files via upload
Ver. 1.1 Added stitching vias to ground.
Other:
- board text added: "Bird Feeder Board Rev 1.1"
- board text removed: "Bird Feeder Board Rev 1.0"
Changed lines of the file:
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@@
 <text x="3.81" y="16.51" size="1.016" layer="27">GND</text>
 <text x="3.81" y="26.67" size="1.016" layer="27">V_BATT</text>
-<text x="34.29" y="2.54" size="1.016" layer="25">Bird Feeder Board Rev 1.0</text>
+<text x="34.29" y="2.54" size="1.016" layer="25">Bird Feeder Board Rev 1.1</text>
 </plain>
 <attributes>
@@
 <wire x1="15.24" y1="24.45" x2="15.24" y2="25.4" width="0.3048" layer="1"/>
 </signal>
+<signal name="N$1">
+<via x="5.08" y="11.43" extent="1-16" drill="0.35"/>
+</signal>
+<signal name="N$2">
+<via x="21.59" y="11.43" extent="1-16" drill="0.35"/>
+</signal>
+<signal name="N$5">
+<via x="43.18" y="11.43" extent="1-16" drill="0.35"/>
+</signal>
+<signal name="N$7">
+<via x="5.08" y="31.75" extent="1-16" drill="0.35"/>
+</signal>
+<signal name="N$12">
+<via x="44.45" y="30.48" extent="1-16" drill="0.35"/>
+</signal>
+<signal name="N$14">
+<via x="26.67" y="44.45" extent="1-16" drill="0.35"/>
+</signal>
+<signal name="N$15">
+<via x="13.97" y="44.45" extent="1-16" drill="0.35"/>
+</signal>
+<signal name="N$16">
+<via x="50.8" y="44.45" extent="1-16" drill="0.35"/>
+</signal>
+<signal name="N$17">
+<via x="52.07" y="22.86" extent="1-16" drill="0.35"/>
+</signal>
+<signal name="N$18">
+<via x="15.24" y="33.02" extent="1-16" drill="0.35"/>
+</signal>
+<signal name="N$19">
+<via x="34.29" y="34.29" extent="1-16" drill="0.35"/>
+</signal>
+<signal name="N$20">
+<via x="33.02" y="20.32" extent="1-16" drill="0.35"/>
+</signal>
+<signal name="N$22">
+<via x="39.37" y="39.37" extent="1-16" drill="0.35"/>
+</signal>
+<signal name="N$23">
+<via x="29.21" y="12.7" extent="1-16" drill="0.35"/>
+</signal>
+<signal name="N$24">
+<via x="46.99" y="20.32" extent="1-16" drill="0.35"/>
+</signal>
 </signals>

Commit message: Add files via upload
Connections:
- net N$10 renamed FSNS_OUT
- net N$13 renamed MIC_OP2
- net N$4 renamed FSNS_OP3
- net N$6 renamed SERV_OUT
- net N$8 renamed FSNS_OP2
- net N$9 renamed MIC_OP3
Routing:
- net 7.4V: track 66.2 -> 61.2 mm
- net GND: vias 12 -> 27
Other:
- board text added: "Bird Feeder Board Rev 1.2"
- board text removed: "Bird Feeder Board Rev 1.1"
Changed lines of the file:
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@@
 <text x="3.81" y="16.51" size="1.016" layer="27">GND</text>
 <text x="3.81" y="26.67" size="1.016" layer="27">V_BATT</text>
-<text x="34.29" y="2.54" size="1.016" layer="25">Bird Feeder Board Rev 1.1</text>
+<text x="34.29" y="2.54" size="1.016" layer="25">Bird Feeder Board Rev 1.2</text>
 </plain>
 <attributes>
@@
 <wire x1="4.55" y1="19.32" x2="6.08" y2="19.32" width="0.3048" layer="1"/>
 <wire x1="6.08" y1="19.32" x2="6.35" y2="19.05" width="0.3048" layer="1"/>
+<via x="3.81" y="12.7" extent="1-16" drill="0.35"/>
+<via x="21.59" y="11.43" extent="1-16" drill="0.35"/>
+<via x="29.21" y="12.7" extent="1-16" drill="0.35"/>
+<via x="43.18" y="11.43" extent="1-16" drill="0.35"/>
+<via x="52.07" y="22.86" extent="1-16" drill="0.35"/>
+<via x="46.99" y="20.32" extent="1-16" drill="0.35"/>
+<via x="33.02" y="20.32" extent="1-16" drill="0.35"/>
+<via x="5.08" y="31.75" extent="1-16" drill="0.35"/>
+<via x="15.24" y="33.02" extent="1-16" drill="0.35"/>
+<via x="44.45" y="30.48" extent="1-16" drill="0.35"/>
+<via x="34.29" y="34.29" extent="1-16" drill="0.35"/>
+<via x="50.8" y="44.45" extent="1-16" drill="0.35"/>
+<via x="39.37" y="39.37" extent="1-16" drill="0.35"/>
+<via x="26.67" y="44.45" extent="1-16" drill="0.35"/>
+<via x="13.97" y="44.45" extent="1-16" drill="0.35"/>
 </signal>
 <signal name="7.4V">
@@
 <wire x1="2.54" y1="21.59" x2="2.54" y2="26.67" width="1.27" layer="1"/>
 <wire x1="49.53" y1="26.67" x2="50.8" y2="27.94" width="1.27" layer="16"/>
-<wire x1="2.54" y1="26.67" x2="48.26" y2="26.67" width="1.27" layer="16"/>
-<wire x1="48.26" y1="26.67" x2="49.53" y2="26.67" width="1.27" layer="16"/>
-<wire x1="48.26" y1="26.67" x2="48.26" y2="21.59" width="1.27" layer="16"/>
+<wire x1="2.54" y1="26.67" x2="43.18" y2="26.67" width="1.27" layer="16"/>
+<wire x1="49.53" y1="26.67" x2="43.18" y2="26.67" width="1.27" layer="16"/>
 <via x="48.26" y="21.59" extent="1-16" drill="0.35"/>
 <wire x1="48.26" y1="21.59" x2="50.8" y2="19.05" width="1.27" layer="1"/>
@@
 <wire x1="4.55" y1="21.32" x2="2.81" y2="21.32" width="0.3048" layer="1"/>
 <wire x1="2.81" y1="21.32" x2="2.54" y2="21.59" width="0.3048" layer="1"/>
+<wire x1="50.8" y1="27.94" x2="48.26" y2="21.59" width="0" layer="19" extent="1-1"/>
 </signal>
 <signal name="MIC_INT" class="2">
@@
 <wire x1="27.94" y1="6.94" x2="28.26" y2="6.62" width="0.3048" layer="1"/>
 </signal>
-<signal name="N$6" class="2">
+<signal name="SERV_OUT" class="2">
 <contactref element="IC1" pad="6"/>
 <wire x1="38.1" y1="31.75" x2="40.64" y2="31.75" width="0.3048" layer="16"/>
@@
 <wire x1="10.16" y1="16.51" x2="24.13" y2="16.51" width="1.27" layer="16"/>
 </signal>
-<signal name="N$9" class="2">
+<signal name="MIC_OP3" class="2">
 <contactref element="IC3" pad="3"/>
 <contactref element="M1" pad="2"/>
@@
 <wire x1="35.56" y1="11.43" x2="35.56" y2="16.51" width="0.3048" layer="1"/>
 </signal>
-<signal name="N$13" class="2">
+<signal name="MIC_OP2" class="2">
 <contactref element="IC3" pad="2"/>
 <contactref element="R5" pad="2"/>
@@
 <wire x1="45.72" y1="13.97" x2="45.72" y2="15.56" width="0.3048" layer="1"/>
 </signal>
-<signal name="N$4" class="2">
+<signal name="FSNS_OP3" class="2">
 <contactref element="FORC_SENS" pad="2"/>
 <contactref element="IC2" pad="3"/>
@@
 <wire x1="20.32" y1="13.97" x2="12.7" y2="6.35" width="0.3048" layer="1"/>
 </signal>
-<signal name="N$10" class="2">
+<signal name="FSNS_OUT" class="2">
 <contactref element="IC2" pad="6"/>
 <contactref element="IC1" pad="3"/>
@@
 <wire x1="35.56" y1="36.83" x2="30.48" y2="36.83" width="0.3048" layer="16"/>
 </signal>
-<signal name="N$8" class="2">
+<signal name="FSNS_OP2" class="2">
 <contactref element="IC2" pad="2"/>
 <contactref element="R1" pad="1"/>
@@
 <wire x1="15.24" y1="24.45" x2="15.24" y2="25.4" width="0.3048" layer="1"/>
 </signal>
-<signal name="N$1">
-<via x="5.08" y="11.43" extent="1-16" drill="0.35"/>
-</signal>
-<signal name="N$2">
-<via x="21.59" y="11.43" extent="1-16" drill="0.35"/>
-</signal>
-<signal name="N$5">
-<via x="43.18" y="11.43" extent="1-16" drill="0.35"/>
-</signal>
-<signal name="N$7">
-<via x="5.08" y="31.75" extent="1-16" drill="0.35"/>
-</signal>
-<signal name="N$12">
-<via x="44.45" y="30.48" extent="1-16" drill="0.35"/>
-</signal>
-<signal name="N$14">
-<via x="26.67" y="44.45" extent="1-16" drill="0.35"/>
-</signal>
-<signal name="N$15">
-<via x="13.97" y="44.45" extent="1-16" drill="0.35"/>
-</signal>
-<signal name="N$16">
-<via x="50.8" y="44.45" extent="1-16" drill="0.35"/>
-</signal>
-<signal name="N$17">
-<via x="52.07" y="22.86" extent="1-16" drill="0.35"/>
-</signal>
-<signal name="N$18">
-<via x="15.24" y="33.02" extent="1-16" drill="0.35"/>
-</signal>
-<signal name="N$19">
-<via x="34.29" y="34.29" extent="1-16" drill="0.35"/>
-</signal>
-<signal name="N$20">
-<via x="33.02" y="20.32" extent="1-16" drill="0.35"/>
-</signal>
-<signal name="N$22">
-<via x="39.37" y="39.37" extent="1-16" drill="0.35"/>
-</signal>
-<signal name="N$23">
-<via x="29.21" y="12.7" extent="1-16" drill="0.35"/>
-</signal>
-<signal name="N$24">
-<via x="46.99" y="20.32" extent="1-16" drill="0.35"/>
-</signal>
 </signals>

Commit message: Add files via upload
Parts:
- added ISP1: AVRISP-6, adafruit:AVRISP
- moved C2 7.62 mm to (44.5, 25.4)
- moved IC2 6.35 mm to (11.4, 29.2)
- moved IC1 5.68 mm to (29.2, 30.5)
- moved M2 5.39 mm to (34.3, 40.6)
- moved C1 3.81 mm to (50.8, 12.7)
- moved C4 3.81 mm to (42.8, 35.8)
- moved R5 3.81 mm to (45.7, 12.7)
- moved R6 3.81 mm to (41.9, 12.7)
- moved FORC_SENS 3.81 mm to (11.4, 6.35)
- moved R2 3.81 mm to (22.9, 10.2)
- moved R4 3.81 mm to (19.1, 15.2)
- moved M1 3.81 mm to (29.2, 3.81)
- moved C5 3.81 mm to (41.9, 19.1)
- moved CN1 3.81 mm to (6.35, 16.5)
- moved IC3 3.81 mm to (34.3, 16.5)
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Connections:
- new net MOSI: IC1.5, ISP1.4
- new net SCK: IC1.7, ISP1.3
- net +5V: now also ISP1.2
- net GND: now also ISP1.6
- net MIC_OUT: now also ISP1.5
- net SERV_OUT: now also ISP1.1
Routing:
- net MOSI: track 0.00 -> 36.2 mm, vias 0 -> 2
- net GND: track 158.5 -> 174.2 mm
- net MIC_OUT: track 27.1 -> 36.4 mm
- net +5V: track 136.5 -> 144.9 mm
- net SCK: track 0.00 -> 6.13 mm
- net 7.4V: track 61.2 -> 66.5 mm, vias 2 -> 1
- net SERV_OUT: track 17.8 -> 21.7 mm, vias 2 -> 1
- net MIC_INT: track 30.3 -> 33.7 mm, vias 1 -> 2
- net FSNS_OP3: track 29.6 -> 31.7 mm
- net FSNS_OUT: track 17.8 -> 18.3 mm
Other:
- board size 160 x 100 mm -> 54.6 x 43.2 mm
- board text added: "Bird Feeder Board Rev 1.3"
- board text removed: "Bird Feeder Board Rev 1.2"
